File: hardware/0.4-w/keyboard.kicad_sch (KiCad schematic)
At the start: 312 parts, among them J1 SWD, J2 USB_C_Receptacle_USB2.0, J3 JST_PH2, J4 Spare IO, Q1 2N7002, Q2 AO3401A, Q3 AO3401A, SW1 RESET, U1 nRF52840_holyiot_18010, U2 SN74LVC1T45DBV, U3 XC6206P332MR, U4 SRV05-4, U5 TP4057

Commit message: 0.4 delete USB and add connector to Unified Daughterboard
Parts:
- removed C1, C10, C11, C12, C13, C14, C15, C16, C17, C18, C19, C2, C20, C23, C27, C3, C4, C5, C6, C7, C8, C9: 100n, Capacitor_SMD:C_0603_1608Metric, symbol Device:C
- removed C24: 10u, Capacitor_SMD:C_0603_1608Metric, symbol Device:C
- removed D1, D2, D3, D4: SK6812-MINI-E, josh-led:SK8612-MINI-E, symbol josh-led:SK6812-MINI-E
- removed D10, D11, D12, D13, D14, D15, D16, D17, D18, D19, D20, D5, D6, D7, D8, D9: WS2812C, josh-led:LED_WS2812B_PLCC4_5.0x5.0mm_P3.2mm, symbol LED:WS2812B
- removed F1: 500mA, josh-passives-smt:Fuse_0805_2012Metric, symbol Device:Polyfuse
- removed J2: USB_C_Receptacle_USB2.0, josh-connectors:USB_C_Receptacle_HRO_TYPE-C-31-M-12, symbol Connector:USB_C_Receptacle_USB2.0
- removed Q1: 2N7002, Package_TO_SOT_SMD:SOT-23, symbol Device:Q_NMOS_GSD
- removed Q2: AO3401A, Package_TO_SOT_SMD:SOT-23, symbol Transistor_FET:AO3401A
- removed R3, R4, R6, R7: 5K1, Resistor_SMD:R_0603_1608Metric, symbol Device:R
- removed U2: SN74LVC1T45DBV, Package_TO_SOT_SMD:SOT-363_SC-70-6, symbol Logic_LevelTranslator:SN74LVC1T45DBV
- removed U4: SRV05-4, Package_TO_SOT_SMD:SOT-23-6, symbol Power_Protection:SRV05-4
- added J?: Spare IO, josh-connectors:4_PIN_THT_Staggered, symbol Connector:Conn_01x04_Male
- renumbered C25 to C2, C26 to C3, C22 to C4, C21 to C5, D21 to D1, D23 to D10, D24 to D11, D22 to D20, D_103 to D_1, D_58 to D_10, D_85 to D_100, D_79 to D_101, D_72 to D_102, D_61 to D_103, D_50 to D_104, D_40 to D_105, D_30 to D_106, D_26 to D_107, D_19 to D_108, D_14 to D_109, D_53 to D_11, D_9 to D_110, D_5 to D_111, D_47 to D_12, D_42 to D_13, D_36 to D_14, D_31 to D_15, D_24 to D_16, D_18 to D_17, D_13 to D_18, D_8 to D_19, D_109 to D_2, D_1 to D_20, D_110 to D_21, D_104 to D_22, D_96 to D_23, D_88 to D_24, D_87 to D_25, D_81 to D_26, D_76 to D_27, D_70 to D_28, D_65 to D_29, D_99 to D_3, D_59 to D_30, D_54 to D_31, D_48 to D_32, D_43 to D_33, D_37 to D_34, D_32 to D_35, D_25 to D_36, D_20 to D_37, D_17 to D_38, D_7 to D_39, D_93 to D_4, D_2 to D_40, D_105 to D_41, D_100 to D_42, D_94 to D_43, D_91 to D_44, D_84 to D_45, D_78 to D_46, D_73 to D_47, D_67 to D_48, D_62 to D_49, D_86 to D_5, D_56 to D_50, D_45 to D_52, D_39 to D_53, D_34 to D_54, D_28 to D_55, D_22 to D_56, D_16 to D_57, D_11 to D_58, D_3 to D_59, D_80 to D_6, D_106 to D_60, D_101 to D_61, D_95 to D_62, D_92 to D_63, D_83 to D_64, D_77 to D_65, D_71 to D_66, D_66 to D_67, D_60 to D_68, D_55 to D_69, D_75 to D_7, D_49 to D_70, D_44 to D_71, D_38 to D_72, D_33 to D_73, D_27 to D_74, D_21 to D_75, D_12 to D_76, D_4 to D_77, D_108 to D_78, D_102 to D_79, D_69 to D_8, D_97 to D_80, D_90 to D_81, D_74 to D_83, D_68 to D_84, D_63 to D_85, D_57 to D_86, D_52 to D_87, D_46 to D_88, D_41 to D_89, D_64 to D_9, D_35 to D_90, D_29 to D_91, D_23 to D_92, D_15 to D_93, D_10 to D_94, D_6 to D_95, D_111 to D_96, D_107 to D_97, D_89 to D_99, J3 to J1, J4 to J3, J1 to J4, JP2 to JP1, JP1 to JP2, K_28 to K_1, K_79 to K_10, K_8 to K_100, K_27 to K_101, K_66 to K_102, K_86 to K_103, K_100 to K_104, K_30 to K_105, K_36 to K_106, K_43 to K_107, K_7 to K_108, K_14 to K_109, K_84 to K_11, K_20 to K_110, K_21 to K_111, K_54 to K_112, K_64 to K_113, K_76 to K_114, K_88 to K_115, K_93 to K_116, K_97 to K_117, K_105 to K_118, K_112 to K_119, K_91 to K_12, K_118 to K_120, K_98 to K_13, K_103 to K_14, K_109 to K_15, K_113 to K_16, K_1 to K_17, K_9 to K_18, K_15 to K_19, K_34 to K_2, K_22 to K_20, K_110 to K_21, K_2 to K_22, K_10 to K_23, K_16 to K_24, K_23 to K_25, K_29 to K_26, K_35 to K_27, K_40 to K_28, K_46 to K_29, K_39 to K_3, K_51 to K_30, K_57 to K_31, K_62 to K_32, K_69 to K_33, K_74 to K_34, K_80 to K_35, K_85 to K_36, K_92 to K_37, K_99 to K_38, K_104 to K_39, K_45 to K_4, K_107 to K_40, K_114 to K_41, K_3 to K_42, K_11 to K_43, K_17 to K_44, K_24 to K_45, K_31 to K_46, K_37 to K_47, K_42 to K_48, K_48 to K_49, K_50 to K_5, K_53 to K_50, K_59 to K_51, K_65 to K_52, K_71 to K_53, K_77 to K_54, K_82 to K_55, K_89 to K_56, K_95 to K_57, K_101 to K_58, K_108 to K_59, K_56 to K_6, K_115 to K_60, K_5 to K_61, K_4 to K_62, K_12 to K_63, K_18 to K_64, K_25 to K_65, K_32 to K_66, K_38 to K_67, K_44 to K_68, K_49 to K_69, K_61 to K_7, K_55 to K_70, K_60 to K_71, K_67 to K_72, K_72 to K_73, K_78 to K_74, K_83 to K_75, K_90 to K_76, K_96 to K_77, K_106 to K_78, K_116 to K_79, K_68 to K_8, K_6 to K_80, K_13 to K_81, K_19 to K_82, K_26 to K_83, K_33 to K_84, K_41 to K_85, K_47 to K_86, K_52 to K_87, K_58 to K_88, K_63 to K_89, K_73 to K_9, K_70 to K_90, K_75 to K_91, K_81 to K_92, K_87 to K_93, K_102 to K_95, K_111 to K_96, K_117 to K_97, K_120 to K_98, K_121 to K_99, LOGO2 to LOGO1, LOGO1 to LOGO2, Q3 to Q2, R11 to R10, R2 to R11, R8 to R5, R10 to R6, R5 to R7, R9 to R8, R1 to R9, U5 to U1, U3 to U2, U1 to U4
Connections:
- net +5V: now also J?.4 (Pin_4)
- net GND: now also J?.1 (Pin_1)
- net USB_D+: now also J?.2 (Pin_2)
- net USB_D-: now also J?.3 (Pin_3)
- no-connect marks 7 -> 2
Other:
- note removed: "3v3 -> VBATT logic shift"
- note removed: "High Side Disable"
- note removed: "Status LEDs"
- note removed: "USB"
- note removed: "Underglow LEDs"
- moved on the sheet: JP1, JP2
